Commit message: update sensor orientation

File: environment_description/urdf/ur5_ft.urdf.xacro (robot description, xacro)
@@ -8,5 +8,5 @@
   <xacro:ur5_robot prefix="" />
   <xacro:robotiq_ft300 parent="tool0" prefix="">
-    <origin xyz="0 0 0" rpy="0 0 0"/>
+    <origin xyz="0 0 0" rpy="0 0 -1.5447"/>
   </xacro:robotiq_ft300>
   <!-- <xacro:robotiq_arg2f_85  prefix="" /> -->
